File: pcb/Xpander6-VIC.brd (EAGLE design)
At the start: 169.9 x 356.9 mm, 59 parts, among them SW11 TL46WO, SW14 TL46WO, SW17 TL46WO, SW3 !RESET, SW6 TL46WO, SW9 TL46WO, X1 FE22-2R, X2 FE22-2R, X3 FE22-2R, X4 MA22-2SHORT, X5 FE22-2R, X6 FE22-2R, X7 FE22-2R

Commit message: Convert 6 slot design to use newer symbols
Parts:
- removed EC1: MA-44, con-edge-156:MA-44
- removed RP1, RP11, RP3, RP5, RP7, RP9: 10K, resistor-net:RN-8
- removed RP10, RP12, RP2, RP4, RP6, RP8: (no value), resistor-net:RN-5
- removed SJ1, SJ2: (no value), jumper:SJ
- removed SW1, SW10, SW13, SW16, SW4, SW7: (no value), special:EDG-08
- removed SW12, SW15, SW18, SW2, SW5, SW8: (no value), special:EDG-04
- removed X1, X2, X3, X5, X6, X7: FE22-2R, con-edge-156:FE22-2_REV
- removed X4: MA22-2SHORT, con-edge-156:MA22-2SHORT
- added AUDIO: (no value), jumper:SJ
- added RN1, RN10, RN12, RN4, RN6, RN8: (no value), resistor-net-rp:RN-7
- added RN11, RN2, RN3, RN5, RN7, RN9: (no value), resistor-net-rp:RN-5
- added S1, S2, S3, S4, S5, S6: (no value), switch-dil-rp:DIP08SB
- added S10, S11, S12, S7, S8, S9: (no value), switch-dil-rp:DIP04SB
- added X10, X11, X12, X13, X14, X9: PORT_EXPANSION_VIC_CONN, commodore:FE156-22-2
- added X16: PORT_EXPANSION_VIC_CONNR, commodore:MA156-22-2SHORT
- added X8: PORT_EXPANSION_VIC_EDGE, commodore:MA156-22-2
- moved SW3 5.24 mm to (124.5, 275.6)
- moved LED1 5.08 mm to (114.9, 0.00)
- moved LED2 5.08 mm to (114.9, 49.5)
- moved LED3 5.08 mm to (114.9, 247.7)
- moved LED4 5.08 mm to (114.9, 99.1)
- moved LED5 5.08 mm to (114.9, 148.6)
- moved LED6 5.08 mm to (114.9, 198.1)
- moved R1 5.08 mm to (116.2, -7.62)
- moved R2 5.08 mm to (116.2, 41.9)
- moved R3 5.08 mm to (116.2, 240.0)
- moved R4 5.08 mm to (116.2, 91.4)
- moved R5 5.08 mm to (116.2, 141.0)
- moved R6 5.08 mm to (116.2, 190.5)
- moved SW11 5.08 mm to (125.7, 99.1)
- moved SW14 5.08 mm to (125.7, 148.6)
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Connections:
- removed net 10: EC1.10, SW1.5, SW10.5, SW13.5, SW16.5, SW4.5, SW7.5
- removed net 11: EC1.11, SW1.6, SW10.6, SW13.6, SW16.6, SW4.6, SW7.6
- removed net 12: EC1.12, SW1.7, SW10.7, SW13.7, SW16.7, SW4.7, SW7.7
- removed net 13: EC1.13, SW1.8, SW10.8, SW13.8, SW16.8, SW4.8, SW7.8
- removed net 14: EC1.14, SW12.1, SW15.1, SW18.1, SW2.1, SW5.1, SW8.1
- removed net 15: EC1.15, SW12.2, SW15.2, SW18.2, SW2.2, SW5.2, SW8.2
- removed net 16: EC1.16, SW12.3, SW15.3, SW18.3, SW2.3, SW5.3, SW8.3
- removed net 17: EC1.17, X1.17, X2.17, X3.17, X4.17, X5.17, X6.17, X7.17
- removed net 18: EC1.18, X1.18, X2.18, X3.18, X4.18, X5.18, X6.18, X7.18
- removed net 19: EC1.19, X1.19, X2.19, X3.19, X4.19, X5.19, X6.19, X7.19
- removed net 2: EC1.2, X1.2, X2.2, X3.2, X4.2, X5.2, X6.2, X7.2
- removed net 20: EC1.20, SJ1.1, SJ1.2, X1.20, X2.20, X3.20, X4.20, X5.20, X6.20, X7.20
- removed net 21: EC1.21, F1.P$2
- removed net 3: EC1.3, X1.3, X2.3, X3.3, X4.3, X5.3, X6.3, X7.3
- removed net 4: EC1.4, X1.4, X2.4, X3.4, X4.4, X5.4, X6.4, X7.4
- removed net 5: EC1.5, X1.5, X2.5, X3.5, X4.5, X5.5, X6.5, X7.5
- removed net 6: EC1.6, X1.6, X2.6, X3.6, X4.6, X5.6, X6.6, X7.6
- removed net 7: EC1.7, X1.7, X2.7, X3.7, X4.7, X5.7, X6.7, X7.7
- removed net 8: EC1.8, X1.8, X2.8, X3.8, X4.8, X5.8, X6.8, X7.8
- removed net 9: EC1.9, X1.9, X2.9, X3.9, X4.9, X5.9, X6.9, X7.9
- removed net B: EC1.B, X1.B, X2.B, X3.B, X4.B, X5.B, X6.B, X7.B
- removed net C: EC1.C, X1.C, X2.C, X3.C, X4.C, X5.C, X6.C, X7.C
- removed net D: EC1.D, X1.D, X2.D, X3.D, X4.D, X5.D, X6.D, X7.D
- removed net E: EC1.E, X1.E, X2.E, X3.E, X4.E, X5.E, X6.E, X7.E
- removed net F: EC1.F, X1.F, X2.F, X3.F, X4.F, X5.F, X6.F, X7.F
- removed net H: EC1.H, X1.H, X2.H, X3.H, X4.H, X5.H, X6.H, X7.H
- removed net J: EC1.J, X1.J, X2.J, X3.J, X4.J, X5.J, X6.J, X7.J
- removed net K: EC1.K, X1.K, X2.K, X3.K, X4.K, X5.K, X6.K, X7.K
- removed net L: EC1.L, X1.L, X2.L, X3.L, X4.L, X5.L, X6.L, X7.L
- removed net M: EC1.M, X1.M, X2.M, X3.M, X4.M, X5.M, X6.M, X7.M
- removed net N: EC1.N, X1.N, X2.N, X3.N, X4.N, X5.N, X6.N, X7.N
- removed net N$1: RP1.5, SW1.12, X1.10
- removed net N$10: RP3.7, SW4.10, X2.12
- removed net N$11: RP6.2, SW8.8, X3.14, X4.14
- removed net N$12: RP3.4, SW4.13, SW6.3, SW6.4
- removed net N$13: RP3.3, SW4.14, SW6.1, SW6.6
- removed net N$14: RP6.3, SW8.7, X3.15, X4.15
- removed net N$15: RP3.8, SW4.9, X2.13
- removed net N$16: RP3.6, SW4.11, X2.11
- removed net N$18: RP5.4, SW7.13, SW9.3, SW9.4
- removed net N$19: SW6.5, X2.T
- removed net N$2: RP1.3, SW1.14, X1.T
- removed net N$20: RP5.7, SW7.10, X3.12, X4.12
- removed net N$21: RP5.8, SW7.9, X3.13, X4.13
- removed net N$22: C3.+, LED3.A, SW7.15, SW7.16, X3.21, X4.21
- removed net N$23: SW6.2, X2.U
- removed net N$24: RP5.3, SW7.14, SW9.1, SW9.6
- removed net N$27: SW9.2, X3.U, X4.U
- removed net N$28: SW9.5, X3.T, X4.T
- removed net N$29: RP5.5, SW7.12, X3.10, X4.10
- removed net N$3: RP1.4, SW1.13, X1.U
- removed net N$30: RP5.6, SW7.11, X3.11, X4.11
- removed net N$31: RP2.2, SW2.8, X1.14
- removed net N$32: RP2.3, SW2.7, X1.15
- removed net N$33: RP2.4, SW2.6, X1.16
- removed net N$34: RP4.2, SW5.8, X2.14
- removed net N$35: RP4.3, SW5.7, X2.15
- removed net N$36: RP4.4, SW5.6, X2.16
- removed net N$37: RP7.4, SW10.13, SW11.3, SW11.4
- removed net N$38: RP7.7, SW10.10, X5.12
- removed net N$39: RP6.4, SW8.6, X3.16, X4.16
- removed net N$4: RP1.6, SW1.11, X1.11
- removed net N$40: RP7.8, SW10.9, X5.13
- removed net N$41: C4.+, LED4.A, SW10.15, SW10.16, X5.21
- removed net N$42: RP7.3, SW10.14, SW11.1, SW11.6
- removed net N$44: SW11.2, X5.U
- removed net N$45: SW11.5, X5.T
- removed net N$46: RP7.5, SW10.12, X5.10
- removed net N$47: RP7.6, SW10.11, X5.11
- removed net N$48: RP8.2, SW12.8, X5.14
- removed net N$49: RP8.3, SW12.7, X5.15
- removed net N$5: RP1.7, SW1.10, X1.12
- removed net N$50: RP8.4, SW12.6, X5.16
- removed net N$51: RP9.4, SW13.13, SW14.3, SW14.4
- removed net N$52: RP9.7, SW13.10, X6.12
- removed net N$53: RP9.8, SW13.9, X6.13
- removed net N$54: C5.+, LED5.A, SW13.15, SW13.16, X6.21
- removed net N$55: RP9.3, SW13.14, SW14.1, SW14.6
- removed net N$57: SW14.2, X6.U
- removed net N$58: SW14.5, X6.T
- removed net N$59: RP9.5, SW13.12, X6.10
- removed net N$6: RP1.8, SW1.9, X1.13
- removed net N$60: RP9.6, SW13.11, X6.11
- removed net N$61: RP10.2, SW15.8, X6.14
- removed net N$62: RP10.3, SW15.7, X6.15
- removed net N$63: RP10.4, SW15.6, X6.16
- removed net N$64: RP11.4, SW16.13, SW17.3, SW17.4
- removed net N$65: RP11.7, SW16.10, X7.12
- removed net N$66: RP11.8, SW16.9, X7.13
- removed net N$67: C6.+, LED6.A, SW16.15, SW16.16, X7.21
- removed net N$68: RP11.3, SW16.14, SW17.1, SW17.6
- removed net N$7: C1.+, LED1.A, SW1.15, SW1.16, X1.21
- removed net N$70: SW17.2, X7.U
- removed net N$71: SW17.5, X7.T
- removed net N$72: RP11.5, SW16.12, X7.10
- removed net N$73: RP11.6, SW16.11, X7.11
- removed net N$74: RP12.2, SW18.8, X7.14
- removed net N$75: RP12.3, SW18.7, X7.15
- removed net N$76: RP12.4, SW18.6, X7.16
- removed net N$8: C2.+, LED2.A, SW4.15, SW4.16, X2.21
- removed net N$9: RP3.5, SW4.12, X2.10
- removed net P: EC1.P, X1.P, X2.P, X3.P, X4.P, X5.P, X6.P, X7.P
- removed net R: EC1.R, X1.R, X2.R, X3.R, X4.R, X5.R, X6.R, X7.R
- removed net S: EC1.S, X1.S, X2.S, X3.S, X4.S, X5.S, X6.S, X7.S
- removed net T: EC1.T, SW1.3, SW10.3, SW13.3, SW16.3, SW4.3, SW7.3
- removed net U: EC1.U, SW1.4, SW10.4, SW13.4, SW16.4, SW4.4, SW7.4
- removed net V: EC1.V, X1.V, X2.V, X3.V, X4.V, X5.V, X6.V, X7.V
- removed net W: EC1.W, X1.W, X2.W, X3.W, X4.W, X5.W, X6.W, X7.W
- removed net X: EC1.X, SW3.2, X1.X, X2.X, X3.X, X4.X, X5.X, X6.X, X7.X
- removed net Y: EC1.Y, SJ2.1, SJ2.2, X1.Y, X2.Y, X3.Y, X4.Y, X5.Y, X6.Y, X7.Y
- new net !BLK1: S1.5, S2.5, S3.5, S4.5, S5.5, S6.5, X8.10
- new net !BLK1_1: RN1.4, S1.12, X9.10
- new net !BLK1_2: RN4.4, S2.12, X10.10
- new net !BLK1_3: RN6.4, S3.12, X11.10
- new net !BLK1_4: RN8.4, S4.12, X12.10
- new net !BLK1_5: RN10.4, S5.12, X13.10
- new net !BLK1_6: RN12.4, S6.12, X14.10, X16.10
- new net !BLK2: S1.6, S2.6, S3.6, S4.6, S5.6, S6.6, X8.11
- new net !BLK2_1: RN1.5, S1.11, X9.11
- new net !BLK2_2: RN4.5, S2.11, X10.11
- new net !BLK2_3: RN6.5, S3.11, X11.11
- new net !BLK2_4: RN8.5, S4.11, X12.11
- new net !BLK2_5: RN10.5, S5.11, X13.11
- new net !BLK2_6: RN12.5, S6.11, X14.11, X16.11
- new net !BLK3: S1.7, S2.7, S3.7, S4.7, S5.7, S6.7, X8.12
- new net !BLK3_1: RN1.6, S1.10, X9.12
- new net !BLK3_2: RN4.6, S2.10, X10.12
- new net !BLK3_3: RN6.6, S3.10, X11.12
- new net !BLK3_4: RN8.6, S4.10, X12.12
- new net !BLK3_5: RN10.6, S5.10, X13.12
- new net !BLK3_6: RN12.6, S6.10, X14.12, X16.12
- new net !BLK5: S1.8, S2.8, S3.8, S4.8, S5.8, S6.8, X8.13
- new net !BLK5_1: RN1.7, S1.9, X9.13
- new net !BLK5_2: RN4.7, S2.9, X10.13
- new net !BLK5_3: RN6.7, S3.9, X11.13
- new net !BLK5_4: RN8.7, S4.9, X12.13
- new net !BLK5_5: RN10.7, S5.9, X13.13
- new net !BLK5_6: RN12.7, S6.9, X14.13, X16.13
- new net !IO2: S1.3, S2.3, S3.3, S4.3, S5.3, S6.3, X8.T
- new net !IO2SW_2: RN4.2, S2.14, SW6.1, SW6.6
- new net !IO2SW_3: RN6.2, S3.14, SW11.1, SW11.6
- new net !IO2SW_4: RN8.2, S4.14, SW14.1, SW14.6
- new net !IO2SW_5: RN10.2, S5.14, SW17.1, SW17.6
- new net !IO2SW_6: RN12.2, S6.14, SW9.1, SW9.6
- new net !IO2_1: RN1.2, S1.14, X9.T
- new net !IO2_2: SW6.5, X10.T
- new net !IO2_3: SW11.5, X11.T
- new net !IO2_4: SW14.5, X12.T
- new net !IO2_5: SW17.5, X13.T
- new net !IO2_6: SW9.5, X14.T, X16.T
- new net !IO3: S1.4, S2.4, S3.4, S4.4, S5.4, S6.4, X8.U
- new net !IO3SW_2: RN4.3, S2.13, SW6.3, SW6.4
- new net !IO3SW_3: RN6.3, S3.13, SW11.3, SW11.4
- new net !IO3SW_4: RN8.3, S4.13, SW14.3, SW14.4
- new net !IO3SW_5: RN10.3, S5.13, SW17.3, SW17.4
- new net !IO3SW_6: RN12.3, S6.13, SW9.3, SW9.4
- new net !IO3_1: RN1.3, S1.13, X9.U
- new net !IO3_2: SW6.2, X10.U
- new net !IO3_3: SW11.2, X11.U
- new net !IO3_4: SW14.2, X12.U
- new net !IO3_5: SW17.2, X13.U
- new net !IO3_6: SW9.2, X14.U, X16.U
- new net !IRQ: X10.19, X11.19, X12.19, X13.19, X14.19, X16.19, X8.19, X9.19
- new net !NMI: X10.W, X11.W, X12.W, X13.W, X14.W, X16.W, X8.W, X9.W
- new net !RAM1: S10.1, S11.1, S12.1, S7.1, S8.1, S9.1, X8.14
- new net !RAM1_1: RN2.2, S7.8, X9.14
- new net !RAM1_2: RN3.2, S8.8, X10.14
- new net !RAM1_3: RN5.2, S9.8, X11.14
- new net !RAM1_4: RN7.2, S10.8, X12.14
- new net !RAM1_5: RN9.2, S11.8, X13.14
- new net !RAM1_6: RN11.2, S12.8, X14.14, X16.14
- new net !RAM2: S10.2, S11.2, S12.2, S7.2, S8.2, S9.2, X8.15
- new net !RAM2_1: RN2.3, S7.7, X9.15
- new net !RAM2_2: RN3.3, S8.7, X10.15
- new net !RAM2_3: RN5.3, S9.7, X11.15
- new net !RAM2_4: RN7.3, S10.7, X12.15
- new net !RAM2_5: RN9.3, S11.7, X13.15
- new net !RAM2_6: RN11.3, S12.7, X14.15, X16.15
- new net !RAM3: S10.3, S11.3, S12.3, S7.3, S8.3, S9.3, X8.16
- new net !RAM3_1: RN2.4, S7.6, X9.16
- new net !RAM3_2: RN3.4, S8.6, X10.16
- new net !RAM3_3: RN5.4, S9.6, X11.16
- new net !RAM3_4: RN7.4, S10.6, X12.16
- new net !RAM3_5: RN9.4, S11.6, X13.16
- new net !RAM3_6: RN11.4, S12.6, X14.16, X16.16
- new net !RESET: SW3.2, X10.X, X11.X, X12.X, X13.X, X14.X, X16.X, X8.X, X9.X
- new net A0: X10.B, X11.B, X12.B, X13.B, X14.B, X16.B, X8.B, X9.B
- new net A1: X10.C, X11.C, X12.C, X13.C, X14.C, X16.C, X8.C, X9.C
- new net A10: X10.N, X11.N, X12.N, X13.N, X14.N, X16.N, X8.N, X9.N
- new net A11: X10.P, X11.P, X12.P, X13.P, X14.P, X16.P, X8.P, X9.P
- new net A12: X10.R, X11.R, X12.R, X13.R, X14.R, X16.R, X8.R, X9.R
- new net A13: X10.S, X11.S, X12.S, X13.S, X14.S, X16.S, X8.S, X9.S
- new net A2: X10.D, X11.D, X12.D, X13.D, X14.D, X16.D, X8.D, X9.D
- new net A3: X10.E, X11.E, X12.E, X13.E, X14.E, X16.E, X8.E, X9.E
- new net A4: X10.F, X11.F, X12.F, X13.F, X14.F, X16.F, X8.F, X9.F
- new net A5: X10.H, X11.H, X12.H, X13.H, X14.H, X16.H, X8.H, X9.H
- new net A6: X10.J, X11.J, X12.J, X13.J, X14.J, X16.J, X8.J, X9.J
- new net A7: X10.K, X11.K, X12.K, X13.K, X14.K, X16.K, X8.K, X9.K
- new net A8: X10.L, X11.L, X12.L, X13.L, X14.L, X16.L, X8.L, X9.L
- new net A9: X10.M, X11.M, X12.M, X13.M, X14.M, X16.M, X8.M, X9.M
- new net AUDIO: AUDIO.1, X8.Y
- new net AUDIO': AUDIO.2, X10.Y, X11.Y, X12.Y, X13.Y, X14.Y, X16.Y, X9.Y
- new net CR/!W: X10.18, X11.18, X12.18, X13.18, X14.18, X16.18, X8.18, X9.18
- new net D0: X10.2, X11.2, X12.2, X13.2, X14.2, X16.2, X8.2, X9.2
- new net D1: X10.3, X11.3, X12.3, X13.3, X14.3, X16.3, X8.3, X9.3
- new net D2: X10.4, X11.4, X12.4, X13.4, X14.4, X16.4, X8.4, X9.4
- new net D3: X10.5, X11.5, X12.5, X13.5, X14.5, X16.5, X8.5, X9.5
- new net D4: X10.6, X11.6, X12.6, X13.6, X14.6, X16.6, X8.6, X9.6
- new net D5: X10.7, X11.7, X12.7, X13.7, X14.7, X16.7, X8.7, X9.7
- new net D6: X10.8, X11.8, X12.8, X13.8, X14.8, X16.8, X8.8, X9.8
- new net D7: X10.9, X11.9, X12.9, X13.9, X14.9, X16.9, X8.9, X9.9
- new net PHI2: X10.V, X11.V, X12.V, X13.V, X14.V, X16.V, X8.V, X9.V
- new net VCC: F1.P$1, X8.21
- new net VCC_1: C1.+, LED1.A, S1.15, S1.16, X9.21
- new net VCC_2: C2.+, LED2.A, S2.15, S2.16, X10.21
- new net VCC_3: C4.+, LED4.A, S3.15, S3.16, X11.21
- new net VCC_4: C5.+, LED5.A, S4.15, S4.16, X12.21
- new net VCC_5: C6.+, LED6.A, S5.15, S5.16, X13.21
- new net VCC_6: C3.+, LED3.A, S6.15, S6.16, X14.21, X16.21
- new net VR/!W: X10.17, X11.17, X12.17, X13.17, X14.17, X16.17, X8.17, X9.17
- net FVCC: now also F1.P$2, RN1.1, RN10.1, RN11.1, RN12.1, RN2.1, RN3.1, RN4.1, RN5.1, RN6.1, RN7.1, RN8.1, RN9.1, S1.1, S1.2, S2.1, S2.2, S3.1, S3.2, S4.1, S4.2, S5.1, S5.2, S6.1, S6.2; no longer F1.P$1, RP1.1, RP10.1, RP11.1, RP12.1, RP2.1, RP3.1, RP4.1, RP5.1, RP6.1, RP7.1, RP8.1, RP9.1, SW1.1, SW1.2, SW10.1, SW10.2, SW13.1, SW13.2, SW16.1, SW16.2, SW4.1, SW4.2, SW7.1, SW7.2
- net GND: now also X10.1, X10.22, X10.A, X10.Z, X11.1, X11.22, X11.A, X11.Z, X12.1, X12.22, X12.A, X12.Z, X13.1, X13.22, X13.A, X13.Z, X14.1, X14.22, X14.A, X14.Z, X16.1, X16.22, X16.A, X16.Z, X8.1, X8.22, X8.A, X8.Z, X9.1, X9.22, X9.A, X9.Z; no longer EC1.1, EC1.22, EC1.A, EC1.Z, X1.1, X1.22, X1.A, X1.Z, X2.1, X2.22, X2.A, X2.Z, X3.1, X3.22, X3.A, X3.Z, X4.1, X4.22, X4.A, X4.Z, X5.1, X5.22, X5.A, X5.Z, X6.1, X6.22, X6.A, X6.Z, X7.1, X7.22, X7.A, X7.Z
Routing:
- net !RESET: track 0.00 -> 516.8 mm, vias 0 -> 2
- net X: track 514.2 -> 0.00 mm, vias 2 -> 0
- net !RAM3: track 0.00 -> 424.2 mm, vias 0 -> 2
- net !RAM2: track 0.00 -> 419.5 mm, vias 0 -> 2
- net 16: track 419.2 -> 0.00 mm, vias 2 -> 0
- net 15: track 414.4 -> 0.00 mm, vias 2 -> 0
- net !RAM1: track 0.00 -> 413.7 mm, vias 0 -> 2
- net 14: track 408.6 -> 0.00 mm, vias 2 -> 0
- net !BLK5: track 0.00 -> 405.4 mm, vias 0 -> 2
- net !IO3: track 0.00 -> 405.0 mm, vias 0 -> 1
- net !IO2: track 0.00 -> 401.3 mm, vias 0 -> 1
- net 13: track 400.3 -> 0.00 mm, vias 2 -> 0
- net U: track 399.9 -> 0.00 mm, vias 1 -> 0
- net !BLK3: track 0.00 -> 399.7 mm, vias 0 -> 2
- net T: track 396.3 -> 0.00 mm, vias 1 -> 0
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- added copper zone on layer 1, net VCC_6
- added copper zone on layer 16, net VCC_6
- removed copper zone on layer 1, net N$22
- removed copper zone on layer 16, net N$22
Other:
- board size 169.9 x 356.9 mm -> 175.3 x 355.6 mm

Commit message: Route optional audio line
Parts:
- moved AUDIO 12.3 mm to (-32.7, -61.4), flipped to the bottom, turned to 180 degrees
- moved F1 9.85 mm to (-37.6, -58.4), turned to 90 degrees
- renumbered X10 to X2, X11 to X3, X12 to X4, X13 to X5, X14 to X6, X16 to X7, X9 to X1
Connections:
- new net AUDIO'_1: S7.5, X1.Y
- new net AUDIO'_2: S8.5, X2.Y
- new net AUDIO'_3: S9.5, X3.Y
- new net AUDIO'_4: S10.5, X4.Y
- new net AUDIO'_5: S11.5, X5.Y
- new net AUDIO'_6: S12.5, X6.Y, X7.Y
- net AUDIO': now also S10.4, S11.4, S12.4, S7.4, S8.4, S9.4; no longer X1.Y, X2.Y, X3.Y, X4.Y, X5.Y, X6.Y, X7.Y
Routing:
- net AUDIO'_6: track 0.00 -> 193.4 mm, vias 0 -> 2
- net AUDIO'_5: track 0.00 -> 174.4 mm, vias 0 -> 2
- net AUDIO'_4: track 0.00 -> 174.4 mm, vias 0 -> 2
- net AUDIO'_3: track 0.00 -> 174.4 mm, vias 0 -> 2
- net AUDIO'_2: track 0.00 -> 174.4 mm, vias 0 -> 2
- net AUDIO'_1: track 0.00 -> 165.9 mm
- net AUDIO': track 335.7 -> 423.5 mm
- net VCC: track 24.4 -> 11.5 mm
- net FVCC: track 608.7 -> 620.6 mm
- net AUDIO: track 22.7 -> 12.6 mm, vias 1 -> 0
- net !RAM3: track 424.2 -> 425.7 mm
- net !IO3: track 405.0 -> 406.5 mm
- net !IO2: track 401.3 -> 402.8 mm
- net !BLK5: track 405.4 -> 406.9 mm
- net !BLK3: track 399.7 -> 401.1 mm
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Other:
- board text added: "AUDIO"
