File: pcb/Xpander6-VIC.brd (EAGLE design)
At the start: 175.3 x 355.6 mm, 58 parts, among them SW11 TL46WO, SW14 TL46WO, SW17 TL46WO, SW3 !RESET, SW6 TL46WO, SW9 TL46WO, X1 PORT_EXPANSION_VIC_CONN, X2 PORT_EXPANSION_VIC_CONN, X3 PORT_EXPANSION_VIC_CONN, X4 PORT_EXPANSION_VIC_CONN, X5 PORT_EXPANSION_VIC_CONN, X6 PORT_EXPANSION_VIC_CONN, X7 PORT_EXPANSION_VIC_CONNR, X8 PORT_EXPANSION_VIC_EDGE

Commit message: More updates
Parts:
- removed SW14: TL46WO, switch:TL4XWO
- added SW1: TL46WO, switch:TL4XWO
- RN10, RN12, RN4, RN6, RN8: device resistor-net-rp:RN-7 -> resistor-net-rp:RN-5
- RN11, RN3, RN5, RN7, RN9: device resistor-net-rp:RN-5 -> resistor-net-rp:RN-7
- S11, S7, S9: device switch-dil-rp:DIP04SB -> switch-dil-rp:DIP08SB
- S2, S4, S6: device switch-dil-rp:DIP08SB -> switch-dil-rp:DIP04SB
- SW3: value !RESET -> TL46WO; device switch-omron:B3F-31XX -> switch:TL4XWO
- SW6: value TL46WO -> !RESET; device switch:TL4XWO -> switch-omron:B3F-31XX
- moved SW6 226.1 mm to (124.5, 275.6), turned to 180 degrees
- moved S6 149.6 mm to (105.4, 99.1)
- moved S7 149.6 mm to (87.6, 148.6)
- moved C3 148.6 mm to (-39.4, 81.3)
- moved LED3 148.6 mm to (114.9, 99.1)
- moved SW3 127.0 mm to (125.7, 148.6), turned to 270 degrees
- moved S4 100.6 mm to (105.4, 49.5)
- moved S9 100.6 mm to (87.6, 198.1)
- moved S5 99.1 mm to (87.6, 99.1)
- moved S8 99.1 mm to (105.4, 148.6)
- moved S11 52.6 mm to (87.6, 247.7)
- moved S2 52.6 mm to (105.4, 0.00)
- moved C4 49.5 mm to (-39.4, 130.8)
- moved C5 49.5 mm to (-39.4, 180.3)
- moved C6 49.5 mm to (-39.4, 229.9)
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- renumbered SW11 to SW2, SW17 to SW4, SW9 to SW5
Connections:
- net !BLK1: now also S11.5, S7.5, S9.5; no longer S2.5, S4.5, S6.5
- net !BLK1_2: now also RN3.4, S3.12; no longer RN4.4, S2.12
- net !BLK1_3: now also RN5.4, S5.12; no longer RN6.4, S3.12
- net !BLK1_4: now also RN7.4, S7.12; no longer RN8.4, S4.12
- net !BLK1_5: now also RN9.4, S9.12; no longer RN10.4, S5.12
- net !BLK1_6: now also RN11.4, S11.12; no longer RN12.4, S6.12
- net !BLK2: now also S11.6, S7.6, S9.6; no longer S2.6, S4.6, S6.6
- net !BLK2_2: now also RN3.5, S3.11; no longer RN4.5, S2.11
- net !BLK2_3: now also RN5.5, S5.11; no longer RN6.5, S3.11
- net !BLK2_4: now also RN7.5, S7.11; no longer RN8.5, S4.11
- net !BLK2_5: now also RN9.5, S9.11; no longer RN10.5, S5.11
- net !BLK2_6: now also RN11.5, S11.11; no longer RN12.5, S6.11
- net !BLK3: now also S11.7, S7.7, S9.7; no longer S2.7, S4.7, S6.7
- net !BLK3_2: now also RN3.6, S3.10; no longer RN4.6, S2.10
- net !BLK3_3: now also RN5.6, S5.10; no longer RN6.6, S3.10
- net !BLK3_4: now also RN7.6, S7.10; no longer RN8.6, S4.10
- net !BLK3_5: now also RN9.6, S9.10; no longer RN10.6, S5.10
- net !BLK3_6: now also RN11.6, S11.10; no longer RN12.6, S6.10
- net !BLK5: now also S11.8, S7.8, S9.8; no longer S2.8, S4.8, S6.8
- net !BLK5_2: now also RN3.7, S3.9; no longer RN4.7, S2.9
- net !BLK5_3: now also RN5.7, S5.9; no longer RN6.7, S3.9
- net !BLK5_4: now also RN7.7, S7.9; no longer RN8.7, S4.9
- net !BLK5_5: now also RN9.7, S9.9; no longer RN10.7, S5.9
- net !BLK5_6: now also RN11.7, S11.9; no longer RN12.7, S6.9
- net !IO2: now also S11.3, S7.3, S9.3; no longer S2.3, S4.3, S6.3
- net !IO2SW_2: now also RN3.2, S3.14, SW1.1, SW1.6; no longer RN4.2, S2.14, SW6.1, SW6.6
- net !IO2SW_3: now also RN5.2, S5.14; no longer RN6.2, S3.14
- net !IO2SW_4: now also RN7.2, S7.14, SW3.1, SW3.6; no longer RN8.2, S4.14, SW14.1, SW14.6
- net !IO2SW_5: now also RN9.2, S9.14; no longer RN10.2, S5.14
- net !IO2SW_6: now also RN11.2, S11.14; no longer RN12.2, S6.14
- net !IO2_2: now also SW1.5; no longer SW6.5
- net !IO2_4: now also SW3.5; no longer SW14.5
- net !IO3: now also S11.4, S7.4, S9.4; no longer S2.4, S4.4, S6.4
- net !IO3SW_2: now also RN3.3, S3.13, SW1.3, SW1.4; no longer RN4.3, S2.13, SW6.3, SW6.4
- net !IO3SW_3: now also RN5.3, S5.13; no longer RN6.3, S3.13
- net !IO3SW_4: now also RN7.3, S7.13, SW3.3, SW3.4; no longer RN8.3, S4.13, SW14.3, SW14.4
- net !IO3SW_5: now also RN9.3, S9.13; no longer RN10.3, S5.13
- net !IO3SW_6: now also RN11.3, S11.13; no longer RN12.3, S6.13
- net !IO3_2: now also SW1.2; no longer SW6.2
- net !IO3_4: now also SW3.2; no longer SW14.2
- net !RAM1: now also S2.1, S4.1, S6.1; no longer S11.1, S7.1, S9.1
- net !RAM1_1: now also S2.8; no longer S7.8
- net !RAM1_2: now also RN4.2, S4.8; no longer RN3.2, S8.8
- net !RAM1_3: now also RN6.2, S6.8; no longer RN5.2, S9.8
- net !RAM1_4: now also RN8.2, S8.8; no longer RN7.2, S10.8
- net !RAM1_5: now also RN10.2, S10.8; no longer RN9.2, S11.8
- net !RAM1_6: now also RN12.2; no longer RN11.2
- net !RAM2: now also S2.2, S4.2, S6.2; no longer S11.2, S7.2, S9.2
- net !RAM2_1: now also S2.7; no longer S7.7
- net !RAM2_2: now also RN4.3, S4.7; no longer RN3.3, S8.7
- net !RAM2_3: now also RN6.3, S6.7; no longer RN5.3, S9.7
- net !RAM2_4: now also RN8.3, S8.7; no longer RN7.3, S10.7
- net !RAM2_5: now also RN10.3, S10.7; no longer RN9.3, S11.7
- net !RAM2_6: now also RN12.3; no longer RN11.3
- net !RAM3: now also S2.3, S4.3, S6.3; no longer S11.3, S7.3, S9.3
- net !RAM3_1: now also S2.6; no longer S7.6
- net !RAM3_2: now also RN4.4, S4.6; no longer RN3.4, S8.6
- net !RAM3_3: now also RN6.4, S6.6; no longer RN5.4, S9.6
- net !RAM3_4: now also RN8.4, S8.6; no longer RN7.4, S10.6
- net !RAM3_5: now also RN10.4, S10.6; no longer RN9.4, S11.6
- net !RAM3_6: now also RN12.4; no longer RN11.4
- net !RESET: now also SW6.2; no longer SW3.2
- net AUDIO': now also S2.4, S4.4, S6.4; no longer S11.4, S7.4, S9.4
- net AUDIO'_1: now also S2.5; no longer S7.5
- net AUDIO'_2: now also S4.5; no longer S8.5
- net AUDIO'_3: now also S6.5; no longer S9.5
- net AUDIO'_4: now also S8.5; no longer S10.5
- net AUDIO'_5: now also S10.5; no longer S11.5
- net FVCC: now also S11.1, S11.2, S7.1, S7.2, S9.1, S9.2; no longer S2.1, S2.2, S4.1, S4.2, S6.1, S6.2
- net GND: now also SW6.1; no longer SW3.1
- net N$26: now also LED6.K; no longer LED3.K
- net N$43: now also LED3.K; no longer LED4.K
- net N$56: now also LED4.K; no longer LED5.K
- net N$69: now also LED5.K; no longer LED6.K
- net VCC_2: now also S3.15, S3.16; no longer S2.15, S2.16
- net VCC_3: now also C3.+, LED3.A, S5.15, S5.16; no longer C4.+, LED4.A, S3.15, S3.16
- net VCC_4: now also C4.+, LED4.A, S7.15, S7.16; no longer C5.+, LED5.A, S4.15, S4.16
- net VCC_5: now also C5.+, LED5.A, S9.15, S9.16; no longer C6.+, LED6.A, S5.15, S5.16
- net VCC_6: now also C6.+, LED6.A, S11.15, S11.16; no longer C3.+, LED3.A, S6.15, S6.16
Routing:
- net AUDIO'_5: track 174.4 -> 168.6 mm, vias 2 -> 1
- net AUDIO'_4: track 174.4 -> 168.6 mm, vias 2 -> 1
- net AUDIO'_3: track 174.4 -> 168.6 mm, vias 2 -> 1
- net AUDIO'_2: track 174.4 -> 168.6 mm, vias 2 -> 1
- net AUDIO'_1: track 165.9 -> 162.1 mm
- net !RAM3_1: track 145.3 -> 141.8 mm
- net AUDIO'_6: track 193.4 -> 196.8 mm
- net !RAM2_1: track 137.7 -> 134.5 mm
- net !IO3_6: track 194.2 -> 191.1 mm
- net !IO3_2: track 166.0 -> 162.8 mm
- net !IO3_5: track 166.0 -> 162.8 mm
- net !IO3_4: track 166.0 -> 162.8 mm
- net !IO3_3: track 166.0 -> 162.8 mm
- net !RAM3_6: track 175.4 -> 172.4 mm
- net !RAM3_5: track 143.5 -> 140.5 mm
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