File: pcb/Xpander6-VIC.sch (EAGLE design)
At the start: 59 parts, among them SW11 TL46WO, SW14 TL46WO, SW17 TL46WO, SW3 !RESET, SW6 TL46WO, SW9 TL46WO, X1 FE22-2R, X2 FE22-2R, X3 FE22-2R, X4 MA22-2SHORT, X5 FE22-2R, X6 FE22-2R, X7 FE22-2R

Commit message: Convert 6 slot design to use newer symbols
Parts:
- removed EC1: MA-44, con-edge-156:MA-44
- removed RP1, RP11, RP3, RP5, RP7, RP9: 10K, resistor-net:RNX7
- removed RP10, RP12, RP2, RP4, RP6, RP8: (no value), resistor-net:RNX4
- removed SJ1, SJ2: (no value), jumper:SJ
- removed SW1, SW10, SW13, SW16, SW4, SW7: (no value), special:SW_DIP-8
- removed SW12, SW15, SW18, SW2, SW5, SW8: (no value), special:SW_DIP-4
- removed X1, X2, X3, X5, X6, X7: FE22-2R, con-edge-156:FE22-2R
- removed X4: MA22-2SHORT, con-edge-156:MA22-2SHORT
- added AUDIO: (no value), jumper:SJ
- added RN1, RN10, RN12, RN4, RN6, RN8: (no value), resistor-net-rp:RNX6
- added RN11, RN2, RN3, RN5, RN7, RN9: (no value), resistor-net-rp:RNX4
- added S1, S2, S3, S4, S5, S6: (no value), switch-dil-rp:DIP08SB
- added S10, S11, S12, S7, S8, S9: (no value), switch-dil-rp:DIP04SB
- added X10, X11, X12, X13, X14, X9: PORT_EXPANSION_VIC_CONN, commodore:PORT_EXPANSION_VIC_CONN
- added X16: PORT_EXPANSION_VIC_CONNR, commodore:PORT_EXPANSION_VIC_CONNR
- added X8: PORT_EXPANSION_VIC_EDGE, commodore:PORT_EXPANSION_VIC_EDGE
Connections:
- removed net 10: EC1.10, SW1.5, SW10.5, SW13.5, SW16.5, SW4.5, SW7.5
- removed net 11: EC1.11, SW1.6, SW10.6, SW13.6, SW16.6, SW4.6, SW7.6
- removed net 12: EC1.12, SW1.7, SW10.7, SW13.7, SW16.7, SW4.7, SW7.7
- removed net 13: EC1.13, SW1.8, SW10.8, SW13.8, SW16.8, SW4.8, SW7.8
- removed net 14: EC1.14, SW12.1, SW15.1, SW18.1, SW2.1, SW5.1, SW8.1
- removed net 15: EC1.15, SW12.2, SW15.2, SW18.2, SW2.2, SW5.2, SW8.2
- removed net 16: EC1.16, SW12.3, SW15.3, SW18.3, SW2.3, SW5.3, SW8.3
- removed net 17: EC1.17, X1.17, X2.17, X3.17, X4.17, X5.17, X6.17, X7.17
- removed net 18: EC1.18, X1.18, X2.18, X3.18, X4.18, X5.18, X6.18, X7.18
- removed net 19: EC1.19, X1.19, X2.19, X3.19, X4.19, X5.19, X6.19, X7.19
- removed net 2: EC1.2, X1.2, X2.2, X3.2, X4.2, X5.2, X6.2, X7.2
- removed net 20: EC1.20, SJ1.1, SJ1.2, X1.20, X2.20, X3.20, X4.20, X5.20, X6.20, X7.20
- removed net 21: EC1.21, F1.2
- removed net 3: EC1.3, X1.3, X2.3, X3.3, X4.3, X5.3, X6.3, X7.3
- removed net 4: EC1.4, X1.4, X2.4, X3.4, X4.4, X5.4, X6.4, X7.4
- removed net 5: EC1.5, X1.5, X2.5, X3.5, X4.5, X5.5, X6.5, X7.5
- removed net 6: EC1.6, X1.6, X2.6, X3.6, X4.6, X5.6, X6.6, X7.6
- removed net 7: EC1.7, X1.7, X2.7, X3.7, X4.7, X5.7, X6.7, X7.7
- removed net 8: EC1.8, X1.8, X2.8, X3.8, X4.8, X5.8, X6.8, X7.8
- removed net 9: EC1.9, X1.9, X2.9, X3.9, X4.9, X5.9, X6.9, X7.9
- removed net B: EC1.B, X1.B, X2.B, X3.B, X4.B, X5.B, X6.B, X7.B
- removed net C: EC1.C, X1.C, X2.C, X3.C, X4.C, X5.C, X6.C, X7.C
- removed net D: EC1.D, X1.D, X2.D, X3.D, X4.D, X5.D, X6.D, X7.D
- removed net E: EC1.E, X1.E, X2.E, X3.E, X4.E, X5.E, X6.E, X7.E
- removed net F: EC1.F, X1.F, X2.F, X3.F, X4.F, X5.F, X6.F, X7.F
- removed net H: EC1.H, X1.H, X2.H, X3.H, X4.H, X5.H, X6.H, X7.H
- removed net J: EC1.J, X1.J, X2.J, X3.J, X4.J, X5.J, X6.J, X7.J
- removed net K: EC1.K, X1.K, X2.K, X3.K, X4.K, X5.K, X6.K, X7.K
- removed net L: EC1.L, X1.L, X2.L, X3.L, X4.L, X5.L, X6.L, X7.L
- removed net M: EC1.M, X1.M, X2.M, X3.M, X4.M, X5.M, X6.M, X7.M
- removed net N: EC1.N, X1.N, X2.N, X3.N, X4.N, X5.N, X6.N, X7.N
- removed net N$1: RP1-4.1, SW1.12, X1.10
- removed net N$10: RP3-6.1, SW4.10, X2.12
- removed net N$11: RP6-1.1, SW8.8, X3.14, X4.14
- removed net N$12: RP3-3.1, SW4.13, SW6.O1, SW6.S
- removed net N$13: RP3-2.1, SW4.14, SW6.O, SW6.S1
- removed net N$14: RP6-2.1, SW8.7, X3.15, X4.15
- removed net N$15: RP3-7.1, SW4.9, X2.13
- removed net N$16: RP3-5.1, SW4.11, X2.11
- removed net N$18: RP5-3.1, SW7.13, SW9.O1, SW9.S
- removed net N$19: SW6.P1, X2.T
- removed net N$2: RP1-2.1, SW1.14, X1.T
- removed net N$20: RP5-6.1, SW7.10, X3.12, X4.12
- removed net N$21: RP5-7.1, SW7.9, X3.13, X4.13
- removed net N$22: C3.+, LED3.A, SW7.15, SW7.16, X3.21, X4.21
- removed net N$23: SW6.P, X2.U
- removed net N$24: RP5-2.1, SW7.14, SW9.O, SW9.S1
- removed net N$27: SW9.P, X3.U, X4.U
- removed net N$28: SW9.P1, X3.T, X4.T
- removed net N$29: RP5-4.1, SW7.12, X3.10, X4.10
- removed net N$3: RP1-3.1, SW1.13, X1.U
- removed net N$30: RP5-5.1, SW7.11, X3.11, X4.11
- removed net N$31: RP2-1.1, SW2.8, X1.14
- removed net N$32: RP2-2.1, SW2.7, X1.15
- removed net N$33: RP2-3.1, SW2.6, X1.16
- removed net N$34: RP4-1.1, SW5.8, X2.14
- removed net N$35: RP4-2.1, SW5.7, X2.15
- removed net N$36: RP4-3.1, SW5.6, X2.16
- removed net N$37: RP7-3.1, SW10.13, SW11.O1, SW11.S
- removed net N$38: RP7-6.1, SW10.10, X5.12
- removed net N$39: RP6-3.1, SW8.6, X3.16, X4.16
- removed net N$4: RP1-5.1, SW1.11, X1.11
- removed net N$40: RP7-7.1, SW10.9, X5.13
- removed net N$41: C4.+, LED4.A, SW10.15, SW10.16, X5.21
- removed net N$42: RP7-2.1, SW10.14, SW11.O, SW11.S1
- removed net N$44: SW11.P, X5.U
- removed net N$45: SW11.P1, X5.T
- removed net N$46: RP7-4.1, SW10.12, X5.10
- removed net N$47: RP7-5.1, SW10.11, X5.11
- removed net N$48: RP8-1.1, SW12.8, X5.14
- removed net N$49: RP8-2.1, SW12.7, X5.15
- removed net N$5: RP1-6.1, SW1.10, X1.12
- removed net N$50: RP8-3.1, SW12.6, X5.16
- removed net N$51: RP9-3.1, SW13.13, SW14.O1, SW14.S
- removed net N$52: RP9-6.1, SW13.10, X6.12
- removed net N$53: RP9-7.1, SW13.9, X6.13
- removed net N$54: C5.+, LED5.A, SW13.15, SW13.16, X6.21
- removed net N$55: RP9-2.1, SW13.14, SW14.O, SW14.S1
- removed net N$57: SW14.P, X6.U
- removed net N$58: SW14.P1, X6.T
- removed net N$59: RP9-4.1, SW13.12, X6.10
- removed net N$6: RP1-7.1, SW1.9, X1.13
- removed net N$60: RP9-5.1, SW13.11, X6.11
- removed net N$61: RP10-1.1, SW15.8, X6.14
- removed net N$62: RP10-2.1, SW15.7, X6.15
- removed net N$63: RP10-3.1, SW15.6, X6.16
- removed net N$64: RP11-3.1, SW16.13, SW17.O1, SW17.S
- removed net N$65: RP11-6.1, SW16.10, X7.12
- removed net N$66: RP11-7.1, SW16.9, X7.13
- removed net N$67: C6.+, LED6.A, SW16.15, SW16.16, X7.21
- removed net N$68: RP11-2.1, SW16.14, SW17.O, SW17.S1
- removed net N$7: C1.+, LED1.A, SW1.15, SW1.16, X1.21
- removed net N$70: SW17.P, X7.U
- removed net N$71: SW17.P1, X7.T
- removed net N$72: RP11-4.1, SW16.12, X7.10
- removed net N$73: RP11-5.1, SW16.11, X7.11
- removed net N$74: RP12-1.1, SW18.8, X7.14
- removed net N$75: RP12-2.1, SW18.7, X7.15
- removed net N$76: RP12-3.1, SW18.6, X7.16
- removed net N$8: C2.+, LED2.A, SW4.15, SW4.16, X2.21
- removed net N$9: RP3-4.1, SW4.12, X2.10
- removed net P: EC1.P, X1.P, X2.P, X3.P, X4.P, X5.P, X6.P, X7.P
- removed net R: EC1.R, X1.R, X2.R, X3.R, X4.R, X5.R, X6.R, X7.R
- removed net S: EC1.S, X1.S, X2.S, X3.S, X4.S, X5.S, X6.S, X7.S
- removed net T: EC1.T, SW1.3, SW10.3, SW13.3, SW16.3, SW4.3, SW7.3
- removed net U: EC1.U, SW1.4, SW10.4, SW13.4, SW16.4, SW4.4, SW7.4
- removed net V: EC1.V, X1.V, X2.V, X3.V, X4.V, X5.V, X6.V, X7.V
- removed net W: EC1.W, X1.W, X2.W, X3.W, X4.W, X5.W, X6.W, X7.W
- removed net X: EC1.X, SW3.S, X1.X, X2.X, X3.X, X4.X, X5.X, X6.X, X7.X
- removed net Y: EC1.Y, SJ2.1, SJ2.2, X1.Y, X2.Y, X3.Y, X4.Y, X5.Y, X6.Y, X7.Y
- new net !BLK1: S1-5.1, S2-5.1, S3-5.1, S4-5.1, S5-5.1, S6-5.1, X8G$1.!BLK1
- new net !BLK1_1: RN1-3.1, S1-5.2, X9A.!BLK1
- new net !BLK1_2: RN4-3.1, S2-5.2, X10A.!BLK1
- new net !BLK1_3: RN6-3.1, S3-5.2, X11A.!BLK1
- new net !BLK1_4: RN8-3.1, S4-5.2, X12A.!BLK1
- new net !BLK1_5: RN10-3.1, S5-5.2, X13A.!BLK1
- new net !BLK1_6: RN12-3.1, S6-5.2, X14A.!BLK1, X16A.!BLK1
- new net !BLK2: S1-6.1, S2-6.1, S3-6.1, S4-6.1, S5-6.1, S6-6.1, X8G$1.!BLK2
- new net !BLK2_1: RN1-4.1, S1-6.2, X9A.!BLK2
- new net !BLK2_2: RN4-4.1, S2-6.2, X10A.!BLK2
- new net !BLK2_3: RN6-4.1, S3-6.2, X11A.!BLK2
- new net !BLK2_4: RN8-4.1, S4-6.2, X12A.!BLK2
- new net !BLK2_5: RN10-4.1, S5-6.2, X13A.!BLK2
- new net !BLK2_6: RN12-4.1, S6-6.2, X14A.!BLK2, X16A.!BLK2
- new net !BLK3: S1-7.1, S2-7.1, S3-7.1, S4-7.1, S5-7.1, S6-7.1, X8G$1.!BLK3
- new net !BLK3_1: RN1-5.1, S1-7.2, X9A.!BLK3
- new net !BLK3_2: RN4-5.1, S2-7.2, X10A.!BLK3
- new net !BLK3_3: RN6-5.1, S3-7.2, X11A.!BLK3
- new net !BLK3_4: RN8-5.1, S4-7.2, X12A.!BLK3
- new net !BLK3_5: RN10-5.1, S5-7.2, X13A.!BLK3
- new net !BLK3_6: RN12-5.1, S6-7.2, X14A.!BLK3, X16A.!BLK3
- new net !BLK5: S1-8.1, S2-8.1, S3-8.1, S4-8.1, S5-8.1, S6-8.1, X8G$1.!BLK5
- new net !BLK5_1: RN1-6.1, S1-8.2, X9A.!BLK5
- new net !BLK5_2: RN4-6.1, S2-8.2, X10A.!BLK5
- new net !BLK5_3: RN6-6.1, S3-8.2, X11A.!BLK5
- new net !BLK5_4: RN8-6.1, S4-8.2, X12A.!BLK5
- new net !BLK5_5: RN10-6.1, S5-8.2, X13A.!BLK5
- new net !BLK5_6: RN12-6.1, S6-8.2, X14A.!BLK5, X16A.!BLK5
- new net !IO2: S1-3.1, S2-3.1, S3-3.1, S4-3.1, S5-3.1, S6-3.1, X8G$1.!IO2
- new net !IO2SW_2: RN4-1.1, S2-3.2, SW6.O, SW6.S1
- new net !IO2SW_3: RN6-1.1, S3-3.2, SW11.O, SW11.S1
- new net !IO2SW_4: RN8-1.1, S4-3.2, SW14.O, SW14.S1
- new net !IO2SW_5: RN10-1.1, S5-3.2, SW17.O, SW17.S1
- new net !IO2SW_6: RN12-1.1, S6-3.2, SW9.O, SW9.S1
- new net !IO2_1: RN1-1.1, S1-3.2, X9A.!IO2
- new net !IO2_2: SW6.P1, X10A.!IO2
- new net !IO2_3: SW11.P1, X11A.!IO2
- new net !IO2_4: SW14.P1, X12A.!IO2
- new net !IO2_5: SW17.P1, X13A.!IO2
- new net !IO2_6: SW9.P1, X14A.!IO2, X16A.!IO2
- new net !IO3: S1-4.1, S2-4.1, S3-4.1, S4-4.1, S5-4.1, S6-4.1, X8G$1.!IO3
- new net !IO3SW_2: RN4-2.1, S2-4.2, SW6.O1, SW6.S
- new net !IO3SW_3: RN6-2.1, S3-4.2, SW11.O1, SW11.S
- new net !IO3SW_4: RN8-2.1, S4-4.2, SW14.O1, SW14.S
- new net !IO3SW_5: RN10-2.1, S5-4.2, SW17.O1, SW17.S
- new net !IO3SW_6: RN12-2.1, S6-4.2, SW9.O1, SW9.S
- new net !IO3_1: RN1-2.1, S1-4.2, X9A.!IO3
- new net !IO3_2: SW6.P, X10A.!IO3
- new net !IO3_3: SW11.P, X11A.!IO3
- new net !IO3_4: SW14.P, X12A.!IO3
- new net !IO3_5: SW17.P, X13A.!IO3
- new net !IO3_6: SW9.P, X14A.!IO3, X16A.!IO3
- new net !IRQ: X10A.!IRQ, X11A.!IRQ, X12A.!IRQ, X13A.!IRQ, X14A.!IRQ, X16A.!IRQ, X8G$1.!IRQ, X9A.!IRQ
- new net !NMI: X10A.!NMI, X11A.!NMI, X12A.!NMI, X13A.!NMI, X14A.!NMI, X16A.!NMI, X8G$1.!NMI, X9A.!NMI
- new net !RAM1: S10-1.1, S11-1.1, S12-1.1, S7-1.1, S8-1.1, S9-1.1, X8G$1.!RAM1
- new net !RAM1_1: RN2-1.1, S7-1.2, X9A.!RAM1
- new net !RAM1_2: RN3-1.1, S8-1.2, X10A.!RAM1
- new net !RAM1_3: RN5-1.1, S9-1.2, X11A.!RAM1
- new net !RAM1_4: RN7-1.1, S10-1.2, X12A.!RAM1
- new net !RAM1_5: RN9-1.1, S11-1.2, X13A.!RAM1
- new net !RAM1_6: RN11-1.1, S12-1.2, X14A.!RAM1, X16A.!RAM1
- new net !RAM2: S10-2.1, S11-2.1, S12-2.1, S7-2.1, S8-2.1, S9-2.1, X8G$1.!RAM2
- new net !RAM2_1: RN2-2.1, S7-2.2, X9A.!RAM2
- new net !RAM2_2: RN3-2.1, S8-2.2, X10A.!RAM2
- new net !RAM2_3: RN5-2.1, S9-2.2, X11A.!RAM2
- new net !RAM2_4: RN7-2.1, S10-2.2, X12A.!RAM2
- new net !RAM2_5: RN9-2.1, S11-2.2, X13A.!RAM2
- new net !RAM2_6: RN11-2.1, S12-2.2, X14A.!RAM2, X16A.!RAM2
- new net !RAM3: S10-3.1, S11-3.1, S12-3.1, S7-3.1, S8-3.1, S9-3.1, X8G$1.!RAM3
- new net !RAM3_1: RN2-3.1, S7-3.2, X9A.!RAM3
- new net !RAM3_2: RN3-3.1, S8-3.2, X10A.!RAM3
- new net !RAM3_3: RN5-3.1, S9-3.2, X11A.!RAM3
- new net !RAM3_4: RN7-3.1, S10-3.2, X12A.!RAM3
- new net !RAM3_5: RN9-3.1, S11-3.2, X13A.!RAM3
- new net !RAM3_6: RN11-3.1, S12-3.2, X14A.!RAM3, X16A.!RAM3
- new net !RESET: SW3.S, X10A.!RESET, X11A.!RESET, X12A.!RESET, X13A.!RESET, X14A.!RESET, X16A.!RESET, X8G$1.!RESET, X9A.!RESET
- new net A0: X10A.A0, X11A.A0, X12A.A0, X13A.A0, X14A.A0, X16A.A0, X8G$1.A0, X9A.A0
- new net A1: X10A.A1, X11A.A1, X12A.A1, X13A.A1, X14A.A1, X16A.A1, X8G$1.A1, X9A.A1
- new net A10: X10A.A10, X11A.A10, X12A.A10, X13A.A10, X14A.A10, X16A.A10, X8G$1.A10, X9A.A10
- new net A11: X10A.A11, X11A.A11, X12A.A11, X13A.A11, X14A.A11, X16A.A11, X8G$1.A11, X9A.A11
- new net A12: X10A.A12, X11A.A12, X12A.A12, X13A.A12, X14A.A12, X16A.A12, X8G$1.A12, X9A.A12
- new net A13: X10A.A13, X11A.A13, X12A.A13, X13A.A13, X14A.A13, X16A.A13, X8G$1.A13, X9A.A13
- new net A2: X10A.A2, X11A.A2, X12A.A2, X13A.A2, X14A.A2, X16A.A2, X8G$1.A2, X9A.A2
- new net A3: X10A.A3, X11A.A3, X12A.A3, X13A.A3, X14A.A3, X16A.A3, X8G$1.A3, X9A.A3
- new net A4: X10A.A4, X11A.A4, X12A.A4, X13A.A4, X14A.A4, X16A.A4, X8G$1.A4, X9A.A4
- new net A5: X10A.A5, X11A.A5, X12A.A5, X13A.A5, X14A.A5, X16A.A5, X8G$1.A5, X9A.A5
- new net A6: X10A.A6, X11A.A6, X12A.A6, X13A.A6, X14A.A6, X16A.A6, X8G$1.A6, X9A.A6
- new net A7: X10A.A7, X11A.A7, X12A.A7, X13A.A7, X14A.A7, X16A.A7, X8G$1.A7, X9A.A7
- new net A8: X10A.A8, X11A.A8, X12A.A8, X13A.A8, X14A.A8, X16A.A8, X8G$1.A8, X9A.A8
- new net A9: X10A.A9, X11A.A9, X12A.A9, X13A.A9, X14A.A9, X16A.A9, X8G$1.A9, X9A.A9
- new net AUDIO: AUDIO.1, X8G$1.AUDIO
- new net AUDIO': AUDIO.2, X10A.AUDIO, X11A.AUDIO, X12A.AUDIO, X13A.AUDIO, X14A.AUDIO, X16A.AUDIO, X9A.AUDIO
- new net CR/!W: X10A.CR/!W, X11A.CR/!W, X12A.CR/!W, X13A.CR/!W, X14A.CR/!W, X16A.CR/!W, X8G$1.CR/!W, X9A.CR/!W
- new net D0: X10A.D0, X11A.D0, X12A.D0, X13A.D0, X14A.D0, X16A.D0, X8G$1.D0, X9A.D0
- new net D1: X10A.D1, X11A.D1, X12A.D1, X13A.D1, X14A.D1, X16A.D1, X8G$1.D1, X9A.D1
- new net D2: X10A.D2, X11A.D2, X12A.D2, X13A.D2, X14A.D2, X16A.D2, X8G$1.D2, X9A.D2
- new net D3: X10A.D3, X11A.D3, X12A.D3, X13A.D3, X14A.D3, X16A.D3, X8G$1.D3, X9A.D3
- new net D4: X10A.D4, X11A.D4, X12A.D4, X13A.D4, X14A.D4, X16A.D4, X8G$1.D4, X9A.D4
- new net D5: X10A.D5, X11A.D5, X12A.D5, X13A.D5, X14A.D5, X16A.D5, X8G$1.D5, X9A.D5
- new net D6: X10A.D6, X11A.D6, X12A.D6, X13A.D6, X14A.D6, X16A.D6, X8G$1.D6, X9A.D6
- new net D7: X10A.D7, X11A.D7, X12A.D7, X13A.D7, X14A.D7, X16A.D7, X8G$1.D7, X9A.D7
- new net PHI2: X10A.PHI2, X11A.PHI2, X12A.PHI2, X13A.PHI2, X14A.PHI2, X16A.PHI2, X8G$1.PHI2, X9A.PHI2
- new net VCC: F1.1, X8G$2.VCC
- new net VCC_1: C1.+, LED1.A, S1-1.2, S1-2.2, X9P.VCC
- new net VCC_2: C2.+, LED2.A, S2-1.2, S2-2.2, X10P.VCC
- new net VCC_3: C4.+, LED4.A, S3-1.2, S3-2.2, X11P.VCC
- new net VCC_4: C5.+, LED5.A, S4-1.2, S4-2.2, X12P.VCC
- new net VCC_5: C6.+, LED6.A, S5-1.2, S5-2.2, X13P.VCC
- new net VCC_6: C3.+, LED3.A, S6-1.2, S6-2.2, X14P.VCC, X16P.VCC
- new net VR/!W: X10A.VR/!W, X11A.VR/!W, X12A.VR/!W, X13A.VR/!W, X14A.VR/!W, X16A.VR/!W, X8G$1.VR/!W, X9A.VR/!W
- net FVCC: now also F1.2, RN10_.1, RN11_.1, RN12_.1, RN1_.1, RN2_.1, RN3_.1, RN4_.1, RN5_.1, RN6_.1, RN7_.1, RN8_.1, RN9_.1, S1-1.1, S1-2.1, S2-1.1, S2-2.1, S3-1.1, S3-2.1, S4-1.1, S4-2.1, S5-1.1, S5-2.1, S6-1.1, S6-2.1; no longer F1.1, RP10_.1, RP11_.1, RP12_.1, RP1_.1, RP2_.1, RP3_.1, RP4_.1, RP5_.1, RP6_.1, RP7_.1, RP8_.1, RP9_.1, SW1.1, SW1.2, SW10.1, SW10.2, SW13.1, SW13.2, SW16.1, SW16.2, SW4.1, SW4.2, SW7.1, SW7.2
- net GND: now also X10P.GND, X10P.GND@1, X10P.GND@2, X10P.GND@3, X11P.GND, X11P.GND@1, X11P.GND@2, X11P.GND@3, X12P.GND, X12P.GND@1, X12P.GND@2, X12P.GND@3, X13P.GND, X13P.GND@1, X13P.GND@2, X13P.GND@3, X14P.GND, X14P.GND@1, X14P.GND@2, X14P.GND@3, X16P.GND, X16P.GND@1, X16P.GND@2, X16P.GND@3, X8G$2.GND, X8G$2.GND@1, X8G$2.GND@2, X8G$2.GND@3, X9P.GND, X9P.GND@1, X9P.GND@2, X9P.GND@3; no longer EC1.1, EC1.22, EC1.A, EC1.Z, X1.1, X1.22, X1.A, X1.Z, X2.1, X2.22, X2.A, X2.Z, X3.1, X3.22, X3.A, X3.Z, X4.1, X4.22, X4.A, X4.Z, X5.1, X5.22, X5.A, X5.Z, X6.1, X6.22, X6.A, X6.Z, X7.1, X7.22, X7.A, X7.Z
Other:
- moved on the sheet: C1, C2, C3, C4, C5, C6, F1, LED1, LED2, LED3, LED4, LED5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

Commit message: Route optional audio line
Parts:
- renumbered X10 to X2, X11 to X3, X12 to X4, X13 to X5, X14 to X6, X16 to X7, X9 to X1
Connections:
- new net AUDIO'_1: S7-4.2, X1A.AUDIO
- new net AUDIO'_2: S8-4.2, X2A.AUDIO
- new net AUDIO'_3: S9-4.2, X3A.AUDIO
- new net AUDIO'_4: S10-4.2, X4A.AUDIO
- new net AUDIO'_5: S11-4.2, X5A.AUDIO
- new net AUDIO'_6: S12-4.2, X6A.AUDIO, X7A.AUDIO
- net AUDIO': now also S10-4.1, S11-4.1, S12-4.1, S7-4.1, S8-4.1, S9-4.1; no longer X1A.AUDIO, X2A.AUDIO, X3A.AUDIO, X4A.AUDIO, X5A.AUDIO, X6A.AUDIO, X7A.AUDIO

Commit message: More updates
Parts:
- removed SW14: TL46WO, switch:TL46WO
- added SW1: TL46WO, switch:TL46WO
- RN10, RN12, RN4, RN6, RN8: device resistor-net-rp:RNX6 -> resistor-net-rp:RNX4
- RN11, RN3, RN5, RN7, RN9: device resistor-net-rp:RNX4 -> resistor-net-rp:RNX6
- S11, S7, S9: device switch-dil-rp:DIP04SB -> switch-dil-rp:DIP08SB
- S2, S4, S6: device switch-dil-rp:DIP08SB -> switch-dil-rp:DIP04SB
- SW3: value !RESET -> TL46WO; device switch-omron:31-XX -> switch:TL46WO
- SW6: value TL46WO -> !RESET; device switch:TL46WO -> switch-omron:31-XX
- renumbered SW11 to SW2, SW17 to SW4, SW9 to SW5
Connections:
- net !BLK1: now also S11-5.1, S7-5.1, S9-5.1; no longer S2-5.1, S4-5.1, S6-5.1
- net !BLK1_2: now also RN3-3.1, S3-5.2; no longer RN4-3.1, S2-5.2
- net !BLK1_3: now also RN5-3.1, S5-5.2; no longer RN6-3.1, S3-5.2
- net !BLK1_4: now also RN7-3.1, S7-5.2; no longer RN8-3.1, S4-5.2
- net !BLK1_5: now also RN9-3.1, S9-5.2; no longer RN10-3.1, S5-5.2
- net !BLK1_6: now also RN11-3.1, S11-5.2; no longer RN12-3.1, S6-5.2
- net !BLK2: now also S11-6.1, S7-6.1, S9-6.1; no longer S2-6.1, S4-6.1, S6-6.1
- net !BLK2_2: now also RN3-4.1, S3-6.2; no longer RN4-4.1, S2-6.2
- net !BLK2_3: now also RN5-4.1, S5-6.2; no longer RN6-4.1, S3-6.2
- net !BLK2_4: now also RN7-4.1, S7-6.2; no longer RN8-4.1, S4-6.2
- net !BLK2_5: now also RN9-4.1, S9-6.2; no longer RN10-4.1, S5-6.2
- net !BLK2_6: now also RN11-4.1, S11-6.2; no longer RN12-4.1, S6-6.2
- net !BLK3: now also S11-7.1, S7-7.1, S9-7.1; no longer S2-7.1, S4-7.1, S6-7.1
- net !BLK3_2: now also RN3-5.1, S3-7.2; no longer RN4-5.1, S2-7.2
- net !BLK3_3: now also RN5-5.1, S5-7.2; no longer RN6-5.1, S3-7.2
- net !BLK3_4: now also RN7-5.1, S7-7.2; no longer RN8-5.1, S4-7.2
- net !BLK3_5: now also RN9-5.1, S9-7.2; no longer RN10-5.1, S5-7.2
- net !BLK3_6: now also RN11-5.1, S11-7.2; no longer RN12-5.1, S6-7.2
- net !BLK5: now also S11-8.1, S7-8.1, S9-8.1; no longer S2-8.1, S4-8.1, S6-8.1
- net !BLK5_2: now also RN3-6.1, S3-8.2; no longer RN4-6.1, S2-8.2
- net !BLK5_3: now also RN5-6.1, S5-8.2; no longer RN6-6.1, S3-8.2
- net !BLK5_4: now also RN7-6.1, S7-8.2; no longer RN8-6.1, S4-8.2
- net !BLK5_5: now also RN9-6.1, S9-8.2; no longer RN10-6.1, S5-8.2
- net !BLK5_6: now also RN11-6.1, S11-8.2; no longer RN12-6.1, S6-8.2
- net !IO2: now also S11-3.1, S7-3.1, S9-3.1; no longer S2-3.1, S4-3.1, S6-3.1
- net !IO2SW_2: now also RN3-1.1, S3-3.2, SW1.O, SW1.S1; no longer RN4-1.1, S2-3.2, SW6.O, SW6.S1
- net !IO2SW_3: now also RN5-1.1, S5-3.2; no longer RN6-1.1, S3-3.2
- net !IO2SW_4: now also RN7-1.1, S7-3.2, SW3.O, SW3.S1; no longer RN8-1.1, S4-3.2, SW14.O, SW14.S1
- net !IO2SW_5: now also RN9-1.1, S9-3.2; no longer RN10-1.1, S5-3.2
- net !IO2SW_6: now also RN11-1.1, S11-3.2; no longer RN12-1.1, S6-3.2
- net !IO2_2: now also SW1.P1; no longer SW6.P1
- net !IO2_4: now also SW3.P1; no longer SW14.P1
- net !IO3: now also S11-4.1, S7-4.1, S9-4.1; no longer S2-4.1, S4-4.1, S6-4.1
- net !IO3SW_2: now also RN3-2.1, S3-4.2, SW1.O1, SW1.S; no longer RN4-2.1, S2-4.2, SW6.O1, SW6.S
- net !IO3SW_3: now also RN5-2.1, S5-4.2; no longer RN6-2.1, S3-4.2
- net !IO3SW_4: now also RN7-2.1, S7-4.2, SW3.O1, SW3.S; no longer RN8-2.1, S4-4.2, SW14.O1, SW14.S
- net !IO3SW_5: now also RN9-2.1, S9-4.2; no longer RN10-2.1, S5-4.2
- net !IO3SW_6: now also RN11-2.1, S11-4.2; no longer RN12-2.1, S6-4.2
- net !IO3_2: now also SW1.P; no longer SW6.P
- net !IO3_4: now also SW3.P; no longer SW14.P
- net !RAM1: now also S2-1.1, S4-1.1, S6-1.1; no longer S11-1.1, S7-1.1, S9-1.1
- net !RAM1_1: now also S2-1.2; no longer S7-1.2
- net !RAM1_2: now also RN4-1.1, S4-1.2; no longer RN3-1.1, S8-1.2
- net !RAM1_3: now also RN6-1.1, S6-1.2; no longer RN5-1.1, S9-1.2
- net !RAM1_4: now also RN8-1.1, S8-1.2; no longer RN7-1.1, S10-1.2
- net !RAM1_5: now also RN10-1.1, S10-1.2; no longer RN9-1.1, S11-1.2
- net !RAM1_6: now also RN12-1.1; no longer RN11-1.1
- net !RAM2: now also S2-2.1, S4-2.1, S6-2.1; no longer S11-2.1, S7-2.1, S9-2.1
- net !RAM2_1: now also S2-2.2; no longer S7-2.2
- net !RAM2_2: now also RN4-2.1, S4-2.2; no longer RN3-2.1, S8-2.2
- net !RAM2_3: now also RN6-2.1, S6-2.2; no longer RN5-2.1, S9-2.2
- net !RAM2_4: now also RN8-2.1, S8-2.2; no longer RN7-2.1, S10-2.2
- net !RAM2_5: now also RN10-2.1, S10-2.2; no longer RN9-2.1, S11-2.2
- net !RAM2_6: now also RN12-2.1; no longer RN11-2.1
- net !RAM3: now also S2-3.1, S4-3.1, S6-3.1; no longer S11-3.1, S7-3.1, S9-3.1
- net !RAM3_1: now also S2-3.2; no longer S7-3.2
- net !RAM3_2: now also RN4-3.1, S4-3.2; no longer RN3-3.1, S8-3.2
- net !RAM3_3: now also RN6-3.1, S6-3.2; no longer RN5-3.1, S9-3.2
- net !RAM3_4: now also RN8-3.1, S8-3.2; no longer RN7-3.1, S10-3.2
- net !RAM3_5: now also RN10-3.1, S10-3.2; no longer RN9-3.1, S11-3.2
- net !RAM3_6: now also RN12-3.1; no longer RN11-3.1
- net !RESET: now also SW6.S; no longer SW3.S
- net AUDIO': now also S2-4.1, S4-4.1, S6-4.1; no longer S11-4.1, S7-4.1, S9-4.1
- net AUDIO'_1: now also S2-4.2; no longer S7-4.2
- net AUDIO'_2: now also S4-4.2; no longer S8-4.2
- net AUDIO'_3: now also S6-4.2; no longer S9-4.2
- net AUDIO'_4: now also S8-4.2; no longer S10-4.2
- net AUDIO'_5: now also S10-4.2; no longer S11-4.2
- net FVCC: now also S11-1.1, S11-2.1, S7-1.1, S7-2.1, S9-1.1, S9-2.1; no longer S2-1.1, S2-2.1, S4-1.1, S4-2.1, S6-1.1, S6-2.1
- net GND: now also SW6.P; no longer SW3.P
- net N$26: now also LED6.C; no longer LED3.C
- net N$43: now also LED3.C; no longer LED4.C
- net N$56: now also LED4.C; no longer LED5.C
- net N$69: now also LED5.C; no longer LED6.C
- net VCC_2: now also S3-1.2, S3-2.2; no longer S2-1.2, S2-2.2
- net VCC_3: now also C3.+, LED3.A, S5-1.2, S5-2.2; no longer C4.+, LED4.A, S3-1.2, S3-2.2
- net VCC_4: now also C4.+, LED4.A, S7-1.2, S7-2.2; no longer C5.+, LED5.A, S4-1.2, S4-2.2
- net VCC_5: now also C5.+, LED5.A, S9-1.2, S9-2.2; no longer C6.+, LED6.A, S5-1.2, S5-2.2
- net VCC_6: now also C6.+, LED6.A, S11-1.2, S11-2.2; no longer C3.+, LED3.A, S6-1.2, S6-2.2
Other:
- moved on the sheet: C3, C4, C5, C6, LED3, LED4, LED5, LED6, RN10-1, RN10-2, RN10-3, RN10-4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
